File: PCB/CAD/Portable-Logger_Dev_101/L70RE.kicad_sch (KiCad schematic)
At the start: 17 parts, among them J1 Conn_Coaxial, Q2 MMBT3904, U1 L76-M33

Commit message: Board Updates
Parts:
- removed U1: L76-M33, GPS L76-M33:L76_QWS, symbol L76L-M33 GNSS:L76-M33
- added U1: L76-M33, RF_GPS:Quectel_L76, symbol GPS_L76:L76-M33
Connections:
- net !GPS_RX: now also U1.3 (RXD1)
- net !GPS_TX: now also U1.2 (TXD1)
- net 1PPS: now also U1.4 (1PPS)
- net 3v3_VCC: now also U1.8 (VCC)
- net GND: now also U1.1 (GND), U1.10 (GND), U1.12 (GND)
- net VBAT_2032: now also U1.6 (V_BCKP)
- net at C14.1, R18.1: now also U1.14 (VCC_REF)
- net at J1.1 (In), L1.2: now also U1.11 (RF_IN)
- net at R17.2: now also U1.9 (RESET)
Changed lines of the file:
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@@
+	)
+	(junction
+		(at 158.75 121.92)
+		(diameter 0)
+		(color 0 0 0 0)
 	)
 	(junction
@@
 	)
 	(junction
-		(at 158.75 121.92)
+		(at 158.75 116.84)
 		(diameter 0)
 		(color 0 0 0 0)
@@
 		(color 0 0 0 0)
 	)
-	(junction
-		(at 158.75 116.84)
-		(diameter 0)
-		(color 0 0 0 0)
-	)
 	(no_connect
 		(at 161.29 106.68)
@@
 	(wire
 		(pts
+			(xy 158.75 121.92) (xy 190.5 121.92)
+		)
+		(stroke
+			(width 0)
+			(type default)
+		)
+	)
+	(wire
+		(pts
 			(xy 166.37 128.27) (xy 157.48 128.27)
 		)
@@
 		(pts
 			(xy 228.6 20.32) (xy 228.6 24.13)
-		)
-		(stroke
-			(width 0)
-			(type default)
-		)
-	)
-	(wire
-		(pts
-			(xy 158.75 121.92) (xy 190.5 121.92)
 		)
 		(stroke
@@
 	)
 	(symbol
-		(lib_id "L76L-M33 GNSS:L76-M33")
+		(lib_id "GPS_L76:L76-M33")
 		(at 87.63 101.6 0)
 		(unit 1)
@@
 			)
 		)
-		(property "Footprint" "GPS L76-M33:L76_QWS"
+		(property "Footprint" "RF_GPS:Quectel_L76"
 			(at 87.63 101.6 0)
 			(effects
@@
 			)
 		)
+		(pin "1"
+		)
+		(pin "6"
+		)
+		(pin "7"
+		)
+		(pin "18"
+		)
+		(pin "8"
+		)
+		(pin "2"
+		)
+		(pin "4"
+		)
+		(pin "3"
+		)
+		(pin "5"
+		)
+		(pin "9"
+		)
+		(pin "12"
+		)
+		(pin "15"
+		)
+		(pin "17"
+		)
+		(pin "13"
+		)
+		(pin "10"
+		)
+		(pin "11"
+		)
 		(pin "16"
 		)
-		(pin "15"
-		)
-		(pin "5"
-		)
-		(pin "2"
-		)
-		(pin "3"
-		)
-		(pin "4"
-		)
-		(pin "6"
-		)
-		(pin "7"
-		)
-		(pin "8"
-		)
-		(pin "1"
-		)
-		(pin "9"
-		)
-		(pin "18"
-		)
-		(pin "17"
-		)
-		(pin "12"
-		)
-		(pin "13"
-		)
-		(pin "11"
-		)
-		(pin "10"
-		)
 		(pin "14"
