File: PCB/CAD/Portable-Logger_Dev_101/Portable-Logger_Dev_101.kicad_sch (KiCad schematic)
At the start: 4 parts, among them U2 ESP32-C6-WROOM-1

Commit message: Board Updates
Parts:
- removed U2: ESP32-C6-WROOM-1, ESPRESSIF footprints:ESP32-C6-WROOM-1, symbol Espressif:ESP32-C6-WROOM-1
- added U3: ESP32-C3-MINI-1, Espressif:ESP32-C3-MINI-1U, symbol Espressif:ESP32-C3-MINI-1
Connections:
- net 3v3_VCC: now also U3.3 (3V3)
- net EN: now also U3.8 (EN/CHIP_PU)
- new net: U3.1 (GND), U3.11 (GND), U3.14 (GND), U3.2 (GND), U3.36 (GND), U3.37 (GND), U3.38 (GND), U3.39 (GND), U3.40 (GND), U3.41 (GND), U3.42 (GND), U3.43 (GND), U3.44 (GND), U3.45 (GND), U3.46 (GND), U3.47 (GND), U3.48 (GND), U3.49 (GND), U3.50 (GND), U3.51 (GND), U3.52 (GND), U3.53 (GND)
- no-connect marks 11 -> 5
