File: PCB/CAD/Logger_Dev_001/_autosave-Logger_Dev_001.kicad_pcb (KiCad board)
At the start: 4 copper layers, 54.5 x 67 mm, 72 parts, among them J1 Conn_Coaxial, J3 Micro_SD_Card_Det1, J4 Connector, USB-TYPE-C-16P, Q1 BC847BS, Q2 MMBT3904, U1 L76-M33, U2 ESP32-C6-WROOM-1, U5 AMS1117, U6 CP2102-GMR

Commit message: Clean PCB and Project
Changed lines of the file:
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@@
+	)
+	(segment
+		(start 149.7 131.075)
+		(end 149.7 131.86)
+		(width 0.5)
+		(layer "F.Cu")
+		(net 1)
 	)
 	(segment
@@
 	)
 	(segment
-		(start 149.55 132.15)
-		(end 149.55 132.01)
-		(width 0.5)
-		(layer "F.Cu")
-		(net 1)
-	)
-	(segment
 		(start 142.775912 130.554088)
 		(end 142.775912 131.54831)
+		(width 0.5)
+		(layer "F.Cu")
+		(net 1)
+	)
+	(segment
+		(start 149.55 132.01)
+		(end 149.55 132.15)
 		(width 0.5)
 		(layer "F.Cu")
@@
 	)
 	(segment
+		(start 149.7 131.86)
+		(end 149.55 132.01)
+		(width 0.5)
+		(layer "F.Cu")
+		(net 1)
+	)
+	(segment
 		(start 164.525 96.375)
 		(end 164.389 96.511)
@@
 	)
 	(segment
-		(start 149.55 132.01)
-		(end 150.24 131.32)
-		(width 0.5)
-		(layer "F.Cu")
-		(net 1)
-	)
-	(segment
 		(start 164.389 96.511)
 		(end 158.536 96.511)
@@
 	)
 	(via
-		(at 150.24 131.32)
+		(at 149.7 131.075)
 		(size 0.8)
 		(drill 0.4)
@@
 	)
 	(segment
-		(start 148.675 93.995)
-		(end 147.435 92.755)
+		(start 148.3 94.9)
+		(end 148.325 94.875)
 		(width 0.2)
 		(layer "F.Cu")
@@
 	)
 	(segment
-		(start 149.057831 95.418493)
-		(end 148.675 95.035662)
+		(start 148.325 94.875)
+		(end 148.325 93.645)
 		(width 0.2)
 		(layer "F.Cu")
@@
 	)
 	(segment
+		(start 147.435 92.755)
+		(end 146.88 92.755)
+		(width 0.2)
+		(layer "F.Cu")
+		(net 18)
+	)
+	(segment
 		(start 136.071855 104.790032)
 		(end 136.046855 104.765032)
@@
 	)
 	(segment
-		(start 147.435 92.755)
-		(end 146.88 92.755)
-		(width 0.2)
-		(layer "F.Cu")
-		(net 18)
-	)
-	(segment
-		(start 149.057831 96.627169)
-		(end 149.057831 95.418493)
+		(start 148.325 93.645)
+		(end 147.435 92.755)
 		(width 0.2)
 		(layer "F.Cu")
@@
 		(start 138.17 105.76)
 		(end 138.17 104.813177)
-		(width 0.2)
-		(layer "F.Cu")
-		(net 18)
-	)
-	(segment
-		(start 148.675 95.035662)
-		(end 148.675 93.995)
 		(width 0.2)
 		(layer "F.Cu")
@@
 	)
 	(via
-		(at 149.057831 96.627169)
+		(at 148.3 94.9)
 		(size 0.7)
 		(drill 0.3)
@@
 	)
 	(segment
-		(start 148.96 100.39)
-		(end 141.225 108.125)
-		(width 0.2)
-		(layer "B.Cu")
-		(net 18)
-	)
-	(segment
-		(start 148.96 96.725)
-		(end 148.96 100.39)
+		(start 148.3 96.065)
+		(end 148.7 96.465)
 		(width 0.2)
 		(layer "B.Cu")
@@
 	)
 	(segment
+		(start 148.3 94.9)
+		(end 148.3 96.065)
+		(width 0.2)
+		(layer "B.Cu")
+		(net 18)
+	)
+	(segment
 		(start 138.17 105.93)
 		(end 138.71 106.47)
@@
 	)
 	(segment
+		(start 148.7 100.65)
+		(end 141.225 108.125)
+		(width 0.2)
+		(layer "B.Cu")
+		(net 18)
+	)
+	(segment
 		(start 138.71 106.47)
 		(end 140.01 106.47)
@@
 	)
 	(segment
-		(start 149.057831 96.627169)
-		(end 148.96 96.725)
-		(width 0.2)
-		(layer "B.Cu")
-		(net 18)
-	)
-	(segment
 		(start 140.01 106.47)
 		(end 141.225 107.685)
@@
 		(start 141.225 107.685)
 		(end 141.225 108.125)
+		(width 0.2)
+		(layer "B.Cu")
+		(net 18)
+	)
+	(segment
+		(start 148.7 96.465)
+		(end 148.7 100.65)
 		(width 0.2)
 		(layer "B.Cu")
@@
 	)
 	(segment
-		(start 151.175 130.4)
+		(start 151 130.225)
 		(end 151.975 131.2)
-		(width 0.2)
-		(layer "F.Cu")
-		(net 26)
-	)
-	(segment
-		(start 148.95 130.4)
-		(end 151.175 130.4)
 		(width 0.2)
 		(layer "F.Cu")
@@
 	)
 	(segment
+		(start 148.1 132.15)
+		(end 148.1 131.25)
+		(width 0.2)
+		(layer "F.Cu")
+		(net 26)
+	)
+	(segment
 		(start 151.975 131.2)
 		(end 151.975 132.675)
@@
 	(segment
 		(start 148.1 131.25)
-		(end 148.95 130.4)
+		(end 149.125 130.225)
 		(width 0.2)
 		(layer "F.Cu")
@@
 	)
 	(segment
-		(start 148.1 132.15)
-		(end 148.1 131.25)
-		(width 0.2)
-		(layer "F.Cu")
+		(start 149.125 130.225)
+		(end 151 130.225)
+		(width 0.2)
+		(layer "F.Cu")
