File: PCB/CAD/Logger_Dev_001/inputUSBto3v3.kicad_sch (KiCad schematic)
At the start: 30 parts, among them J4 Connector, USB-TYPE-C-16P, Q1 BC847BS, U5 AMS1117, U6 CP2102-GMR

Commit message: Clean PCB and Project
Connections:
- net GND: no longer C9.1, J4.S1 (SHIELD)
- new net RF_GND: C9.1, J4.S1 (SHIELD)
Changed lines of the file:
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@@
 	)
 	(junction
-		(at 27.94 78.74)
-		(diameter 0)
-		(color 0 0 0 0)
-	)
-	(junction
 		(at 189.23 67.31)
 		(diameter 0)
@@
 	(wire
 		(pts
-			(xy 27.94 78.74) (xy 27.94 82.55)
-		)
-		(stroke
-			(width 0)
-			(type default)
-		)
-	)
-	(wire
-		(pts
 			(xy 191.77 123.19) (xy 191.77 130.81)
 		)
@@
 	(wire
 		(pts
-			(xy 27.94 72.39) (xy 27.94 78.74)
+			(xy 27.94 72.39) (xy 27.94 82.55)
 		)
 		(stroke
@@
 					(unit 1)
 				)
-			)
-		)
-	)
-	(symbol
-		(lib_name "PWR_FLAG_1")
-		(lib_id "power:PWR_FLAG")
-		(at 27.94 78.74 90)
-		(unit 1)
-		(exclude_from_sim no)
-		(in_bom yes)
-		(on_board yes)
-		(dnp no)
-		(property "Reference" "#FLG03"
-			(at 26.035 78.74 0)
-			(effects
-				(font
-					(size 1.27 1.27)
-				)
-				(hide yes)
-			)
-		)
-		(property "Value" "PWR_FLAG"
-			(at 20.066 78.74 90)
-			(effects
-				(font
-					(size 1.27 1.27)
-				)
-			)
-		)
-		(property "Footprint" ""
-			(at 27.94 78.74 0)
-			(effects
-				(font
-					(size 1.27 1.27)
-				)
-				(hide yes)
-			)
-		)
-		(property "Datasheet" "~"
-			(at 27.94 78.74 0)
-			(effects
-				(font
-					(size 1.27 1.27)
-				)
-				(hide yes)
-			)
-		)
-		(property "Description" "Special symbol for telling ERC where power comes from"
-			(at 27.94 78.74 0)
-			(effects
-				(font
-					(size 1.27 1.27)
-				)
-				(hide yes)
-			)
-		)
-		(pin "1"
-		)
-		(instances
-			(project "Logger_Dev_001"
-				(path "/9546b831-c7ee-4f40-8993-5fd5a38d4078/588c330f-0a28-4ec5-8e7c-c377534893c3"
-					(reference "#FLG03")
-					(unit 1)
-				)
